File: tom-1-clock.sch (KiCad schematic (older format))
At the start: 10 parts, among them U8 LM555xN

Commit message: Next level
Parts:
- added C30: 10uF, Capacitor_THT:C_Disc_D3.0mm_W1.6mm_P2.50mm, symbol Device:CP
- added J2: USB Module, Connector_PinHeader_2.54mm:PinHeader_1x06_P2.54mm_Vertical, symbol Connector_Generic:Conn_01x06
- added Q1: BC517, Package_TO_SOT_THT:TO-92_Inline, symbol Transistor_BJT:BC517
- added R5: 1K, Resistor_THT:R_Axial_DIN0204_L3.6mm_D1.6mm_P1.90mm_Vertical, symbol Device:R
- added R6: 20K, Resistor_THT:R_Axial_DIN0204_L3.6mm_D1.6mm_P1.90mm_Vertical, symbol Device:R
- added R7, R8: R, Resistor_THT:R_Axial_DIN0204_L3.6mm_D1.6mm_P1.90mm_Vertical, symbol Device:R
- added SW1: SW_PUSH, Button_Switch_THT:SW_PUSH_6mm, symbol Switch:SW_Push
- SW2: renamed from Step1; value SW_Push -> SW_PUSH
Connections:
- net VCC: now also J2.1 (Pin_1), R6.1, R8.1
- net CLK renamed clk
- net clk: now also R7.2
- new net: R5.2, SW1.2
- new net: Q1.2 (B), R7.1
- new net GNDREF: C30.2, J2.2 (Pin_2), Q1.3 (E), SW1.1
- new net clk_bar: Q1.1 (C), R8.2
- new net ~Reset: C30.1, R5.1, R6.2
Other:
- note added: "Reset generation"
- moved on the sheet: C1, C2, C3, D1, JP1, R2, R3, R4, SW2, U8

Commit message: Initial commit
Parts:
- added D2: LED, LED_THT:LED_D3.0mm, symbol Device:LED
- added R9: R, Resistor_THT:R_Axial_DIN0204_L3.6mm_D1.6mm_P1.90mm_Vertical, symbol Device:R
Connections:
- net GNDREF: now also R9.2
- net VCC: now also D2.2 (A)
- net clk_bar renamed ~clk
- new net: D2.1 (K), R9.1
Changed lines of the file:
@@
 $EndComp
 Wire Wire Line
-	8550 2100 8100 2100
-Wire Wire Line
-	8550 2200 8100 2200
+	8550 2100 8400 2100
+Wire Wire Line
+	8550 2200 8400 2200
 $Comp
 L power:GNDREF #PWR?
@@
 $EndComp
 Text HLabel 4600 5500 2    50   Output ~ 0
-clk_bar
+~clk
+Wire Wire Line
+	8400 2100 8400 1700
+Wire Wire Line
+	8400 1700 7700 1700
+Wire Wire Line
+	7700 1700 7700 1850
+Wire Wire Line
+	7700 2700 8400 2700
+Wire Wire Line
+	8400 2700 8400 2200
+Connection ~ 8400 2100
+Wire Wire Line
+	8400 2100 8100 2100
+Connection ~ 8400 2200
+Wire Wire Line
+	8400 2200 8100 2200
+$Comp
+L Device:LED D2
+U 1 1 5F1F53C9
+P 7700 2000
+F 0 "D2" V 7739 1882 50  0000 R CNN
+F 1 "LED" V 7648 1882 50  0000 R CNN
+F 2 "LED_THT:LED_D3.0mm" H 7700 2000 50  0001 C CNN
+F 3 "~" H 7700 2000 50  0001 C CNN
+	1    7700 2000
+	0    -1   -1   0
+$EndComp
+Wire Wire Line
+	7700 2150 7700 2300
+$Comp
+L Device:R R9
+U 1 1 5F1F6242
+P 7700 2450
+F 0 "R9" H 7770 2496 50  0000 L CNN
+F 1 "R" H 7770 2405 50  0000 L CNN
+F 2 "Resistor_THT:R_Axial_DIN0204_L3.6mm_D1.6mm_P1.90mm_Vertical" V 7630 2450 50  0001 C CNN
+F 3 "~" H 7700 2450 50  0001 C CNN
+	1    7700 2450
+	1    0    0    -1
+$EndComp
+Wire Wire Line
+	7700 2600 7700 2700
 $EndSCHEMATC
