File: tom-1-dr_registers.sch (KiCad schematic (older format))
At the start: 5 parts, among them IC4 74HC273, J5 Conn_02x08_Top_Bottom, U16 74HC273, U17 74HC273, U6 74HC273

Commit message: Next level
Parts:
- IC4: value 74HC273 -> 74HC697; symbol 74xx:74HC273 -> 74xx:74LS697
- U16, U17, U6: value 74HC273 -> 74LS697; symbol 74xx:74HC273 -> 74xx:74LS697
Connections:
- net labels added: stack[0..7], ~d_enable, ~r_enable
- net labels removed: dr[0..15], r0, r1, r10, r11, r12, r13, r14, r15, r2, r3, r4, r5, r6, r7, r8, r9, stack10, stack11, stack12, stack13, stack14, stack15, stack8, stack9, stack[0..15]
- wire segments 64 -> 60
- no-connect marks 0 -> 18
Other:
- moved on the sheet: IC4, U16, U17, U6

Commit message: Initial commit
Connections:
- net labels added: clk, d_U_~D, d_rck, r_U_~D, r_rck, ~d_output_enable, ~r_output_enable
- wire segments 60 -> 64
Changed lines of the file:
@@
 $Descr A4 11693 8268
 encoding utf-8
-Sheet 10 13
+Sheet 13 13
 Title ""
 Date ""
@@
 	1150 5700 1900 5700
 Wire Wire Line
-	1900 2300 1150 2300
-Wire Wire Line
 	1150 2400 1900 2400
 Wire Wire Line
@@
 Wire Wire Line
 	6000 2350 5550 2350
-Wire Wire Line
-	6000 2250 5550 2250
-Wire Wire Line
-	6000 6150 5550 6150
 Wire Wire Line
 	6000 5550 5550 5550
@@
 stack[0..7]
 Wire Wire Line
-	1250 2800 2000 2800
-Wire Wire Line
 	2000 2900 1250 2900
 Wire Wire Line
-	1900 3000 1150 3000
-Wire Wire Line
 	2000 3350 1250 3350
 Wire Wire Line
 	2000 3450 1250 3450
 Wire Wire Line
-	2000 5900 1250 5900
-Wire Wire Line
-	2000 6000 1250 6000
+	2000 5900 1700 5900
 Wire Wire Line
 	2000 6100 1250 6100
 Wire Wire Line
-	1900 6200 1150 6200
-Wire Wire Line
 	2000 6550 1250 6550
 Wire Wire Line
 	2000 6650 1250 6650
 Wire Wire Line
-	6100 2650 5350 2650
-Wire Wire Line
-	6100 2750 5350 2750
+	6100 2650 5850 2650
 Wire Wire Line
 	6100 2850 5350 2850
 Wire Wire Line
-	6000 2950 5250 2950
-Wire Wire Line
 	6100 3300 5350 3300
 Wire Wire Line
 	6100 3400 5350 3400
 Wire Wire Line
-	6100 5850 5350 5850
-Wire Wire Line
-	6100 5950 5350 5950
+	6100 5850 5800 5850
 Wire Wire Line
 	6100 6050 5350 6050
@@
 NoConn ~ 1900 5000
 Wire Wire Line
-	2000 2700 1150 2700
+	2000 2700 1600 2700
 $Comp
 L power:VCC #PWR0166
 U 1 1 5F0FDEF9
-P 1150 2700
-F 0 "#PWR0166" H 1150 2550 50  0001 C CNN
-F 1 "VCC" H 1165 2873 50  0000 C CNN
-F 2 "" H 1150 2700 50  0001 C CNN
-F 3 "" H 1150 2700 50  0001 C CNN
-	1    1150 2700
+P 1600 2700
+F 0 "#PWR0166" H 1600 2550 50  0001 C CNN
+F 1 "VCC" H 1615 2873 50  0000 C CNN
+F 2 "" H 1600 2700 50  0001 C CNN
+F 3 "" H 1600 2700 50  0001 C CNN
+	1    1600 2700
 	1    0    0    -1
 $EndComp
@@
 L power:VCC #PWR0167
 U 1 1 5F0FE298
-P 1250 5900
-F 0 "#PWR0167" H 1250 5750 50  0001 C CNN
-F 1 "VCC" H 1265 6073 50  0000 C CNN
-F 2 "" H 1250 5900 50  0001 C CNN
-F 3 "" H 1250 5900 50  0001 C CNN
-	1    1250 5900
+P 1700 5900
+F 0 "#PWR0167" H 1700 5750 50  0001 C CNN
+F 1 "VCC" H 1715 6073 50  0000 C CNN
+F 2 "" H 1700 5900 50  0001 C CNN
+F 3 "" H 1700 5900 50  0001 C CNN
+	1    1700 5900
 	1    0    0    -1
 $EndComp
@@
 L power:VCC #PWR0168
 U 1 1 5F0FE874
-P 5350 2650
-F 0 "#PWR0168" H 5350 2500 50  0001 C CNN
-F 1 "VCC" H 5365 2823 50  0000 C CNN
-F 2 "" H 5350 2650 50  0001 C CNN
-F 3 "" H 5350 2650 50  0001 C CNN
-	1    5350 2650
+P 5850 2650
+F 0 "#PWR0168" H 5850 2500 50  0001 C CNN
+F 1 "VCC" H 5865 2823 50  0000 C CNN
+F 2 "" H 5850 2650 50  0001 C CNN
+F 3 "" H 5850 2650 50  0001 C CNN
+	1    5850 2650
 	1    0    0    -1
 $EndComp
@@
 L power:VCC #PWR0169
 U 1 1 5F0FEE02
-P 5350 5850
-F 0 "#PWR0169" H 5350 5700 50  0001 C CNN
-F 1 "VCC" H 5365 6023 50  0000 C CNN
-F 2 "" H 5350 5850 50  0001 C CNN
-F 3 "" H 5350 5850 50  0001 C CNN
-	1    5350 5850
+P 5800 5850
+F 0 "#PWR0169" H 5800 5700 50  0001 C CNN
+F 1 "VCC" H 5815 6023 50  0000 C CNN
+F 2 "" H 5800 5850 50  0001 C CNN
+F 3 "" H 5800 5850 50  0001 C CNN
+	1    5800 5850
 	1    0    0    -1
 $EndComp
@@
 Wire Wire Line
 	5350 3900 5350 5450
+$Comp
+L power:GNDREF #PWR0115
+U 1 1 5ED887FF
+P 5050 2250
+F 0 "#PWR0115" H 5050 2000 50  0001 C CNN
+F 1 "GNDREF" H 5055 2077 50  0000 C CNN
+F 2 "" H 5050 2250 50  0001 C CNN
+F 3 "" H 5050 2250 50  0001 C CNN
+	1    5050 2250
+	1    0    0    -1
+$EndComp
+$Comp
+L power:GNDREF #PWR0116
+U 1 1 5ED88AAD
+P 650 2300
+F 0 "#PWR0116" H 650 2050 50  0001 C CNN
+F 1 "GNDREF" H 655 2127 50  0000 C CNN
+F 2 "" H 650 2300 50  0001 C CNN
+F 3 "" H 650 2300 50  0001 C CNN
+	1    650  2300
+	1    0    0    -1
+$EndComp
+Wire Wire Line
+	650  2300 1900 2300
+Wire Wire Line
+	5050 2250 6000 2250
+Text HLabel 1150 2500 0    50   Input ~ 0
+d_U_~D
+Text HLabel 1150 5700 0    50   Input ~ 0
+d_U_~D
+Text HLabel 5550 2450 0    50   Input ~ 0
+r_U_~D
+Text HLabel 5550 5650 0    50   Input ~ 0
+r_U_~D
+Text HLabel 5350 3300 0    50   Input ~ 0
+clk
+Text HLabel 5350 6500 0    50   Input ~ 0
+clk
+Text HLabel 1250 6550 0    50   Input ~ 0
+clk
+Text HLabel 1250 3350 0    50   Input ~ 0
+clk
+Wire Wire Line
+	2000 2800 1600 2800
+Wire Wire Line
+	6100 2750 5850 2750
+Wire Wire Line
+	6100 5950 5800 5950
+Wire Wire Line
+	2000 6000 1700 6000
+$Comp
+L power:GNDREF #PWR0117
+U 1 1 5ED9D8D2
+P 5850 2750
+F 0 "#PWR0117" H 5850 2500 50  0001 C CNN
+F 1 "GNDREF" H 5855 2577 50  0000 C CNN
+F 2 "" H 5850 2750 50  0001 C CNN
+F 3 "" H 5850 2750 50  0001 C CNN
+	1    5850 2750
+	1    0    0    -1
+$EndComp
+$Comp
+L power:GNDREF #PWR0118
+U 1 1 5ED9DD06
+P 1600 2800
+F 0 "#PWR0118" H 1600 2550 50  0001 C CNN
+F 1 "GNDREF" H 1605 2627 50  0000 C CNN
+F 2 "" H 1600 2800 50  0001 C CNN
+F 3 "" H 1600 2800 50  0001 C CNN
+	1    1600 2800
+	1    0    0    -1
+$EndComp
+$Comp
+L power:GNDREF #PWR0174
+U 1 1 5ED9E060
+P 1700 6000
+F 0 "#PWR0174" H 1700 5750 50  0001 C CNN
+F 1 "GNDREF" H 1705 5827 50  0000 C CNN
+F 2 "" H 1700 6000 50  0001 C CNN
+F 3 "" H 1700 6000 50  0001 C CNN
+	1    1700 6000
+	1    0    0    -1
+$EndComp
+$Comp
+L power:GNDREF #PWR0175
+U 1 1 5ED9E356
+P 5800 5950
+F 0 "#PWR0175" H 5800 5700 50  0001 C CNN
+F 1 "GNDREF" H 5805 5777 50  0000 C CNN
+F 2 "" H 5800 5950 50  0001 C CNN
+F 3 "" H 5800 5950 50  0001 C CNN
+	1    5800 5950
+	1    0    0    -1
+$EndComp
+Text HLabel 1250 3450 0    50   Input ~ 0
+d_rck
+Text HLabel 5350 3400 0    50   Input ~ 0
+r_rck
+Text HLabel 5350 6600 0    50   Input ~ 0
+r_rck
+Text HLabel 1250 6650 0    50   Input ~ 0
+d_rck
+Text HLabel 1250 2900 0    50   Input ~ 0
+~d_output_enable
+Text HLabel 1250 6100 0    50   Input ~ 0
+~d_output_enable
+Text HLabel 5350 2850 0    50   Input ~ 0
+~r_output_enable
+Text HLabel 5350 6050 0    50   Input ~ 0
+~r_output_enable
+Wire Wire Line
+	6000 6150 6000 6350
+Wire Wire Line
+	6000 6350 5550 6350
+Wire Wire Line
+	6000 2950 6000 3200
+Wire Wire Line
+	6000 3200 5500 3200
+Wire Wire Line
+	1900 3000 1900 3250
+Wire Wire Line
+	1900 3250 1550 3250
+Wire Wire Line
+	1900 6200 1900 6450
+Wire Wire Line
+	1900 6450 1550 6450
 Wire Bus Line
 	7700 3300 7700 5500
@@
 Wire Bus Line
 	7700 1050 7700 3300
+$Comp
+L power:VCC #PWR0176
+U 1 1 5EDB0EC1
+P 1550 3250
+F 0 "#PWR0176" H 1550 3100 50  0001 C CNN
+F 1 "VCC" H 1565 3423 50  0000 C CNN
+F 2 "" H 1550 3250 50  0001 C CNN
+F 3 "" H 1550 3250 50  0001 C CNN
+	1    1550 3250
+	1    0    0    -1
+$EndComp
+$Comp
+L power:VCC #PWR0177
+U 1 1 5EDB1284
+P 1550 6450
+F 0 "#PWR0177" H 1550 6300 50  0001 C CNN
+F 1 "VCC" H 1565 6623 50  0000 C CNN
+F 2 "" H 1550 6450 50  0001 C CNN
+F 3 "" H 1550 6450 50  0001 C CNN
+	1    1550 6450
+	1    0    0    -1
+$EndComp
+$Comp
+L power:VCC #PWR0178
+U 1 1 5EDB161C
+P 5550 6350
+F 0 "#PWR0178" H 5550 6200 50  0001 C CNN
+F 1 "VCC" H 5565 6523 50  0000 C CNN
+F 2 "" H 5550 6350 50  0001 C CNN
+F 3 "" H 5550 6350 50  0001 C CNN
+	1    5550 6350
+	1    0    0    -1
+$EndComp
+$Comp
+L power:VCC #PWR0179
+U 1 1 5EDB1CCE
+P 5500 3200
+F 0 "#PWR0179" H 5500 3050 50  0001 C CNN
+F 1 "VCC" H 5515 3373 50  0000 C CNN
+F 2 "" H 5500 3200 50  0001 C CNN
+F 3 "" H 5500 3200 50  0001 C CNN
+	1    5500 3200
+	1    0    0    -1
+$EndComp
 $EndSCHEMATC
