File: tom-1-lcd.sch (KiCad schematic (older format))
At the start: 2 parts, among them U27 KingBright_PSA08-11-MyParts

Commit message: Next level
Other:
- moved on the sheet: R1, U27
Changed lines of the file:
@@
 $Descr A4 11693 8268
 encoding utf-8
-Sheet 3 12
+Sheet 3 13
 Title ""
 Date ""
@@
 L Device:R R1
 U 1 1 5ECAD660
-P 6200 2950
-F 0 "R1" H 6270 2996 50  0000 L CNN
-F 1 "R" H 6270 2905 50  0000 L CNN
-F 2 "Resistor_THT:R_Axial_DIN0204_L3.6mm_D1.6mm_P1.90mm_Vertical" V 6130 2950 50  0001 C CNN
-F 3 "~" H 6200 2950 50  0001 C CNN
-	1    6200 2950
+P 7900 3500
+F 0 "R1" H 7970 3546 50  0000 L CNN
+F 1 "R" H 7970 3455 50  0000 L CNN
+F 2 "Resistor_THT:R_Axial_DIN0204_L3.6mm_D1.6mm_P1.90mm_Vertical" V 7830 3500 50  0001 C CNN
+F 3 "~" H 7900 3500 50  0001 C CNN
+	1    7900 3500
 	0    -1   -1   0
 $EndComp
 Wire Bus Line
-	1200 1250 1850 1250
-Text GLabel 1200 1250 0    50   Input ~ 0
-tos[0..15]
+	2900 2150 3550 2150
 Entry Wire Line
-	1850 1900 1950 2000
+	3550 2450 3650 2550
 Entry Wire Line
-	1850 2000 1950 2100
+	3550 2550 3650 2650
 Entry Wire Line
-	1850 2100 1950 2200
+	3550 2650 3650 2750
 Entry Wire Line
-	1850 2200 1950 2300
+	3550 2750 3650 2850
 Entry Wire Line
-	1850 2300 1950 2400
+	3550 2850 3650 2950
 Entry Wire Line
-	1850 2400 1950 2500
+	3550 2950 3650 3050
 Entry Wire Line
-	1850 2500 1950 2600
+	3550 3050 3650 3150
 Entry Wire Line
-	1850 2600 1950 2700
+	3550 3150 3650 3250
 Entry Wire Line
-	1850 2950 1950 3050
+	3550 3500 3650 3600
 Entry Wire Line
-	1850 3050 1950 3150
+	3550 3600 3650 3700
 Entry Wire Line
-	1850 3150 1950 3250
+	3550 3700 3650 3800
 Entry Wire Line
-	1850 3250 1950 3350
+	3550 3800 3650 3900
 Entry Wire Line
-	1850 3350 1950 3450
+	3550 3900 3650 4000
 Entry Wire Line
-	1850 3450 1950 3550
+	3550 4000 3650 4100
 Entry Wire Line
-	1850 3550 1950 3650
+	3550 4100 3650 4200
 Entry Wire Line
-	1850 3650 1950 3750
-Text GLabel 7000 2950 2    50   Output ~ 0
-jump0
+	3550 4200 3650 4300
 Wire Wire Line
-	6350 2950 7000 2950
+	8050 3500 8700 3500
 Wire Wire Line
-	4550 2600 4300 2600
+	6250 3150 6000 3150
 Wire Wire Line
-	4300 2500 4650 2500
+	6000 3050 6350 3050
 Wire Wire Line
-	4750 2400 4300 2400
+	6450 2950 6000 2950
 Wire Wire Line
-	4300 2300 4850 2300
+	6000 2850 6550 2850
 Wire Wire Line
-	4950 2200 4300 2200
+	6650 2750 6000 2750
 Wire Wire Line
-	4300 2100 5150 2100
+	6000 2650 6850 2650
 Wire Wire Line
-	5250 2000 4300 2000
+	6950 2550 6000 2550
 $Comp
 L Display4x16segment-rescue:KingBright_PSA08-11-MyParts U27
 U 1 1 5EC28090
-P 3650 2400
-F 0 "U27" H 3650 3065 50  0000 C CNN
-F 1 "KingBright_PSA08-11-MyParts" H 3650 2974 50  0000 C CNN
-F 2 "LED_THT:EightSegment" H 3650 2400 50  0001 C CNN
-F 3 "" H 3650 2400 50  0001 C CNN
-	1    3650 2400
+P 5350 2950
+F 0 "U27" H 5350 3615 50  0000 C CNN
+F 1 "KingBright_PSA08-11-MyParts" H 5350 3524 50  0000 C CNN
+F 2 "LED_THT:EightSegment" H 5350 2950 50  0001 C CNN
+F 3 "" H 5350 2950 50  0001 C CNN
+	1    5350 2950
 	1    0    0    -1
 $EndComp
 Wire Wire Line
-	1950 2000 3000 2000
+	3650 2550 4700 2550
 Wire Wire Line
-	1950 2100 3000 2100
+	3650 2650 4700 2650
 Wire Wire Line
-	1950 2200 3000 2200
+	3650 2750 4700 2750
 Wire Wire Line
-	1950 2300 3000 2300
+	3650 2850 4700 2850
 Wire Wire Line
-	1950 2400 3000 2400
+	3650 2950 4700 2950
 Wire Wire Line
-	1950 2500 3000 2500
+	3650 3050 4700 3050
 Wire Wire Line
-	1950 2600 3000 2600
+	3650 3150 4700 3150
 Wire Wire Line
-	1950 2700 3000 2700
+	3650 3250 4700 3250
 Wire Wire Line
-	1950 3050 4450 3050
+	3650 3600 6150 3600
 Wire Wire Line
-	4450 3050 4450 2700
+	6150 3600 6150 3250
 Wire Wire Line
-	4450 2700 4300 2700
+	6150 3250 6000 3250
 Wire Wire Line
-	4550 2600 4550 3150
+	6250 3150 6250 3700
 Wire Wire Line
-	4550 3150 1950 3150
+	6250 3700 3650 3700
 Wire Wire Line
-	1950 3250 4650 3250
+	3650 3800 6350 3800
 Wire Wire Line
-	4650 2500 4650 3250
+	6350 3050 6350 3800
 Wire Wire Line
-	1950 3350 4750 3350
+	3650 3900 6450 3900
 Wire Wire Line
-	4750 2400 4750 3350
+	6450 2950 6450 3900
 Wire Wire Line
-	1950 3450 4850 3450
+	3650 4000 6550 4000
 Wire Wire Line
-	4850 2300 4850 3450
+	6550 2850 6550 4000
 Wire Wire Line
-	1950 3550 4950 3550
+	3650 4100 6650 4100
 Wire Wire Line
-	4950 2200 4950 3550
+	6650 2750 6650 4100
 Wire Wire Line
-	1950 3650 5150 3650
+	3650 4200 6850 4200
 Wire Wire Line
-	5150 2100 5150 3650
+	6850 2650 6850 4200
 Wire Wire Line
-	1950 3750 5250 3750
+	3650 4300 6950 4300
 Wire Wire Line
-	5250 2000 5250 3750
+	6950 2550 6950 4300
 Wire Wire Line
-	3000 2800 2800 2800
+	4700 3350 4500 3350
 Wire Wire Line
-	2800 2800 2800 2950
+	4500 3350 4500 3500
 Wire Wire Line
-	2800 2950 6050 2950
-Text Label 2100 2000 0    50   ~ 0
+	4500 3500 7750 3500
+Text Label 3800 2550 0    50   ~ 0
 tos0
-Text Label 2100 2100 0    50   ~ 0
+Text Label 3800 2650 0    50   ~ 0
 tos1
-Text Label 2100 2200 0    50   ~ 0
+Text Label 3800 2750 0    50   ~ 0
 tos2
-Text Label 2100 2300 0    50   ~ 0
+Text Label 3800 2850 0    50   ~ 0
 tos3
-Text Label 2100 2400 0    50   ~ 0
+Text Label 3800 2950 0    50   ~ 0
 tos4
-Text Label 2100 2500 0    50   ~ 0
+Text Label 3800 3050 0    50   ~ 0
 tos5
-Text Label 2100 2600 0    50   ~ 0
+Text Label 3800 3150 0    50   ~ 0
 tos6
-Text Label 2100 2700 0    50   ~ 0
+Text Label 3800 3250 0    50   ~ 0
 tos7
-Text Label 2100 3050 0    50   ~ 0
+Text Label 3800 3600 0    50   ~ 0
 tos8
-Text Label 2100 3150 0    50   ~ 0
+Text Label 3800 3700 0    50   ~ 0
 tos9
-Text Label 2100 3250 0    50   ~ 0
+Text Label 3800 3800 0    50   ~ 0
 tos10
-Text Label 2100 3350 0    50   ~ 0
+Text Label 3800 3900 0    50   ~ 0
 tos11
-Text Label 2100 3450 0    50   ~ 0
+Text Label 3800 4000 0    50   ~ 0
 tos12
-Text Label 2100 3550 0    50   ~ 0
+Text Label 3800 4100 0    50   ~ 0
 tos13
-Text Label 2100 3650 0    50   ~ 0
+Text Label 3800 4200 0    50   ~ 0
 tos14
-Text Label 2100 3750 0    50   ~ 0
+Text Label 3800 4300 0    50   ~ 0
 tos15
+Text HLabel 2900 2150 0    50   Input ~ 0
+tos[0..15]
+Text HLabel 8700 3500 2    50   Output ~ 0
+jump0
 Wire Bus Line
-	1850 1250 1850 4500
+	3550 2150 3550 4200
 $EndSCHEMATC

Commit message: Initial commit
Connections:
- net jump0 renamed ~jump0
Changed lines of the file:
@@
 tos[0..15]
 Text HLabel 8700 3500 2    50   Output ~ 0
-jump0
+~jump0
 Wire Bus Line
 	3550 2150 3550 4200
