File: tom-1-nand.sch (KiCad schematic (older format))
At the start: 5 parts, among them J4 Conn_02x08_Top_Bottom, U14 74LS00, U15 74LS00, U2 74LS00, U3 74LS00

Commit message: Next level
Connections:
- net labels added: enable
- net labels removed: VCC
- wire segments 57 -> 65
Other:
- moved on the sheet: U14A, U14B, U14C, U14D, U15A, U15B, U15C, U15D, U2A, U2B, U2C, U2D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
