File: tom-1-ram.sch (KiCad schematic (older format))
At the start: 3 parts, among them J6 Conn_02x08_Top_Bottom, U22 CY62256, U28 CY62256

Commit message: Next level
Connections:
- net ~chip_enable~: now reaches U22.20 (~CE)
- net ~output_enable~: now reaches U22.22 (~OE)
- net ~output_enable~: now also U28.22 (~OE)
- net ~write_enable~: now reaches U22.27 (~WE)
- net ~write_enable~: now also U28.27 (~WE)
- net ~chip_enable: now reaches U28.20 (~CE)
Other:
- moved on the sheet: U22, U28
