File: tom-1-rom.sch (KiCad schematic (older format))
At the start: 2 parts, among them J10 Conn_02x08_Top_Bottom, U20 27C1024

Commit message: Next level
Parts:
- added A8: Conn_01x01_Male, Connector_PinHeader_2.54mm:PinHeader_1x01_P2.54mm_Vertical, symbol Connector:Conn_01x01_Male
Connections:
- net ~chip_enable~: now reaches U20.2 (~CE)
- net ~output_enable~: now reaches U20.20 (~OE)
- net at U20.39 (~PGM): now also A8.1 (Pin_1)
Other:
- moved on the sheet: J10, U20

Commit message: Initial commit
Parts:
- renumbered A8 to PGM1
Changed lines of the file:
@@
 	3150 4250 3150 4500
 $Comp
-L Connector:Conn_01x01_Male A8
+L Connector:Conn_01x01_Male PGM1
 U 1 1 5EE65DAF
 P 2950 4500
-F 0 "A8" H 3058 4681 50  0000 C CNN
+F 0 "PGM1" H 3058 4681 50  0000 C CNN
 F 1 "Conn_01x01_Male" H 3058 4590 50  0000 C CNN
 F 2 "Connector_PinHeader_2.54mm:PinHeader_1x01_P2.54mm_Vertical" H 2950 4500 50  0001 C CNN
