File: tom-1-stack.sch (KiCad schematic (older format))
At the start: 3 parts, among them J8 Conn_02x08_Top_Bottom, U10 2KB_SRAM, U11 2KB_SRAM

Commit message: Next level
Connections:
- net stack10 is gone; now on net stack2: U11.6 (A2)
- net stack11 is gone; now on net stack3: U11.5 (A3~)
- net stack12 is gone; now on net stack4: U11.4 (A4~)
- net stack13 is gone; now on net stack5: U11.3 (A5~)
- net stack14 is gone; now on net stack6: U11.2 (A6~)
- net stack15 is gone; now on net stack7: U11.1 (A7)
- net stack8 is gone; now on net stack0: U11.8 (A0)
- net stack9 is gone; now on net stack1: U11.7 (A1)
- net GNDREF: now reaches U10.12 (GND~)
- net GNDREF: now also U11.12 (GND~)
- net VCC: now reaches U10.24 (VCC)
- net VCC: now also U11.24 (VCC)
- net stack_a8 renamed a8
Changed lines of the file:
@@
 $Descr A4 11693 8268
 encoding utf-8
-Sheet 8 12
+Sheet 12 13
 Title ""
 Date ""
@@
 Text Notes 3000 1050 0    50   ~ 0
 STACK: SRAM (2K x 16) with 1.5K unused
-Wire Wire Line
-	4100 1750 4150 1750
 $Comp
 L Connector_Generic:Conn_02x08_Top_Bottom J?
@@
 	1    0    0    -1
 $EndComp
-Entry Wire Line
-	9850 2600 9950 2700
-Entry Wire Line
-	9850 2700 9950 2800
-Entry Wire Line
-	9850 2800 9950 2900
-Entry Wire Line
-	9850 2900 9950 3000
-Entry Wire Line
-	9850 3000 9950 3100
-Entry Wire Line
-	9850 3100 9950 3200
-Entry Wire Line
-	9850 3200 9950 3300
-Entry Wire Line
-	9850 3300 9950 3400
-Entry Wire Line
-	10450 2700 10550 2800
-Entry Wire Line
-	10450 2800 10550 2900
-Entry Wire Line
-	10450 2900 10550 3000
-Entry Wire Line
-	10450 3000 10550 3100
-Entry Wire Line
-	10450 3100 10550 3200
-Entry Wire Line
-	10450 3200 10550 3300
-Entry Wire Line
-	10450 3300 10550 3400
-Entry Wire Line
-	10450 3400 10550 3500
 Wire Bus Line
 	2250 3750 1600 3750
@@
 Entry Wire Line
 	2250 4350 2350 4450
-Text GLabel 1600 3750 0    50   Input ~ 0
-stack[0..15]
-Text GLabel 5850 3750 2    50   Output ~ 0
-stack_bus[0..15]
 Text Label 4600 2450 2    50   ~ 0
 stack_bus7
@@
 stack0
 Text Label 2400 3750 0    50   ~ 0
-stack15
+stack7
 Text Label 2400 3850 0    50   ~ 0
-stack14
+stack6
 Text Label 2400 3950 0    50   ~ 0
-stack13
+stack5
 Text Label 2400 4050 0    50   ~ 0
-stack12
+stack4
 Text Label 2400 4150 0    50   ~ 0
-stack11
+stack3
 Text Label 2400 4250 0    50   ~ 0
-stack10
+stack2
 Text Label 2400 4350 0    50   ~ 0
-stack9
+stack1
 Text Label 2400 4450 0    50   ~ 0
-stack8
+stack0
 Wire Wire Line
 	4150 1850 4550 1850
-Text GLabel 4550 1850 2    50   Output ~ 0
-stack_a8
 Wire Wire Line
 	4150 3850 4550 3850
-Text GLabel 4550 3850 2    50   Output ~ 0
-stack_a8
-Wire Bus Line
-	2250 3750 2250 5650
-Wire Bus Line
-	2250 1550 2250 3750
-Wire Bus Line
-	5200 3750 5200 5650
-Wire Bus Line
-	5200 1500 5200 3750
+Text HLabel 4450 3400 0    50   Input ~ 0
+a8
+Text HLabel 4450 1450 0    50   Input ~ 0
+a8
+Text HLabel 5850 3750 2    50   Output ~ 0
+stack_bus[0..15]
+Text HLabel 1600 3750 0    50   Input ~ 0
+stack[0..7]
+Wire Wire Line
+	4550 3850 4550 3400
+Wire Wire Line
+	4550 3400 4450 3400
+Wire Wire Line
+	4550 1850 4550 1450
+Wire Wire Line
+	4550 1450 4450 1450
+$Comp
+L power:VCC #PWR0170
+U 1 1 5EFF4D1D
+P 4150 1750
+F 0 "#PWR0170" H 4150 1600 50  0001 C CNN
+F 1 "VCC" H 4165 1923 50  0000 C CNN
+F 2 "" H 4150 1750 50  0001 C CNN
+F 3 "" H 4150 1750 50  0001 C CNN
+	1    4150 1750
+	1    0    0    -1
+$EndComp
+$Comp
+L power:GNDREF #PWR0171
+U 1 1 5EFF5019
+P 3350 2850
+F 0 "#PWR0171" H 3350 2600 50  0001 C CNN
+F 1 "GNDREF" H 3355 2677 50  0000 C CNN
+F 2 "" H 3350 2850 50  0001 C CNN
+F 3 "" H 3350 2850 50  0001 C CNN
+	1    3350 2850
+	1    0    0    -1
+$EndComp
+$Comp
+L power:VCC #PWR0172
+U 1 1 5EFF527C
+P 4150 3750
+F 0 "#PWR0172" H 4150 3600 50  0001 C CNN
+F 1 "VCC" H 4165 3923 50  0000 C CNN
+F 2 "" H 4150 3750 50  0001 C CNN
+F 3 "" H 4150 3750 50  0001 C CNN
+	1    4150 3750
+	1    0    0    -1
+$EndComp
+$Comp
+L power:GNDREF #PWR0173
+U 1 1 5EFF559A
+P 3350 4850
+F 0 "#PWR0173" H 3350 4600 50  0001 C CNN
+F 1 "GNDREF" H 3355 4677 50  0000 C CNN
+F 2 "" H 3350 4850 50  0001 C CNN
+F 3 "" H 3350 4850 50  0001 C CNN
+	1    3350 4850
+	1    0    0    -1
+$EndComp
+Wire Bus Line
+	2250 3750 2250 4350
+Wire Bus Line
+	2250 1650 2250 3750
+Wire Bus Line
+	5200 3750 5200 5250
+Wire Bus Line
+	5200 2550 5200 3750
 $EndSCHEMATC

Commit message: Initial commit
Connections:
- net GNDREF: now also U10.19 (A10), U10.22 (A9), U11.19 (A10), U11.22 (A9)
- net ~chip_select: now reaches U10.18 (~CS)
- net ~chip_select: now also U11.18 (~CS)
- net ~output_enable: now reaches U10.20 (~OE)
- net ~output_enable: now also U11.20 (~OE)
- net ~write_enable: now reaches U10.21 (~WE)
- net ~write_enable: now also U11.21 (~WE)
Changed lines of the file:
@@
 $Descr A4 11693 8268
 encoding utf-8
-Sheet 12 13
+Sheet 11 13
 Title ""
 Date ""
@@
 	1    0    0    -1
 $EndComp
+Wire Wire Line
+	4150 1950 4800 1950
+$Comp
+L power:GNDREF #PWR0109
+U 1 1 5ED133B0
+P 4800 2250
+F 0 "#PWR0109" H 4800 2000 50  0001 C CNN
+F 1 "GNDREF" H 4805 2077 50  0000 C CNN
+F 2 "" H 4800 2250 50  0001 C CNN
+F 3 "" H 4800 2250 50  0001 C CNN
+	1    4800 2250
+	1    0    0    -1
+$EndComp
+Wire Wire Line
+	4150 3950 4750 3950
+$Comp
+L power:GNDREF #PWR0110
+U 1 1 5ED14CD4
+P 4750 4250
+F 0 "#PWR0110" H 4750 4000 50  0001 C CNN
+F 1 "GNDREF" H 4755 4077 50  0000 C CNN
+F 2 "" H 4750 4250 50  0001 C CNN
+F 3 "" H 4750 4250 50  0001 C CNN
+	1    4750 4250
+	1    0    0    -1
+$EndComp
+Wire Wire Line
+	4150 2250 4800 2250
+Wire Wire Line
+	4800 2250 4800 1950
+Connection ~ 4800 2250
+Wire Wire Line
+	4750 3950 4750 4250
+Wire Wire Line
+	4750 4250 4150 4250
 Wire Bus Line
 	2250 3750 2250 4350
@@
 Wire Bus Line
 	5200 2550 5200 3750
+Connection ~ 4750 4250
+Text HLabel 4150 2050 2    50   Input ~ 0
+~write_enable
+Text HLabel 4150 4050 2    50   Input ~ 0
+~write_enable
+Text HLabel 4150 4150 2    50   Input ~ 0
+~output_enable
+Text HLabel 4150 2150 2    50   Input ~ 0
+~output_enable
+Text HLabel 4150 2350 2    50   Input ~ 0
+~chip_select
+Text HLabel 4150 4350 2    50   Input ~ 0
+~chip_select
 $EndSCHEMATC
