File: tom-1-tos.sch (KiCad schematic (older format))
At the start: 3 parts, among them IC7 74LS377, IC9 74LS377, J7 Conn_02x08_Top_Bottom

Commit message: Next level
Other:
- moved on the sheet: IC7, IC9, J7

Commit message: Initial commit
Connections:
- net ~clock_enable: now reaches IC7.1 (~E)
- net ~clock_enable: now also IC9.1 (~E)
- net clk: now reaches IC7.11 (CP)
- net clk: now also IC9.11 (CP)
Changed lines of the file:
@@
 Wire Bus Line
 	4800 2050 4800 5250
+Text HLabel 3200 2850 0    50   Input ~ 0
+clk
+Text HLabel 3200 5350 0    50   Input ~ 0
+clk
+Text HLabel 3200 2950 0    50   Input ~ 0
+~clock_enable
+Text HLabel 3200 5450 0    50   Input ~ 0
+~clock_enable
 $EndSCHEMATC
