File: tom-1.kicad_pcb (KiCad board)
At the start: 4 copper layers, 127 x 127 mm, 75 parts, among them IC4 74HC273, IC7 74LS377, IC9 74LS377, J1 Conn_02x06_Counter_Clockwise, J10 Conn_02x08_Top_Bottom, J11 Conn_02x08_Top_Bottom, J2 USB_B_Micro, J3 Conn_02x06_Counter_Clockwise, J4 Conn_02x08_Top_Bottom, J5 Conn_02x08_Top_Bottom, J6 Conn_02x08_Top_Bottom, J7 Conn_02x08_Top_Bottom, J8 Conn_02x08_Top_Bottom, J9 Conn_02x08_Top_Bottom, U1 74LS377, U10 2KB_SRAM, U11 2KB_SRAM, U12 74LS283, U13 74LS283, U14 74LS00, U15 74LS00, U16 74HC273, U17 74HC273, U18 74LS283, U19 74LS283, U2 74LS00, U20 27C1024, U21 74LS193, U22 CY62256, U23 74LS193, U24 74LS193, U25 74LS193, U27 KingBright_PSA08-11-MyParts, U28 CY62256, U3 74LS00, U5 74LS377, U6 74HC273, U8 LM555xN

Commit message: Next level
Parts:
- removed J3: Conn_02x06_Counter_Clockwise, Connector_PinSocket_2.54mm:PinSocket_2x06_P2.54mm_Vertical
- removed Reset1, Step1: SW_Push, Button_Switch_THT:SW_PUSH_6mm
- removed U5: 74LS377, Package_DIP:DIP-20_W7.62mm
- added A8: Conn_01x01_Male, Connector_PinHeader_2.54mm:PinHeader_1x01_P2.54mm_Vertical, F.Cu at (74.7, 21.0)
- added C30: 10uF, Capacitor_THT:C_Disc_D3.0mm_W1.6mm_P2.50mm, F.Cu at (29.0, 128.9)
- added Q1: BC517, Package_TO_SOT_THT:TO-92_Inline, F.Cu at (42.3, 141.6)
- added R5: 1K, Resistor_THT:R_Axial_DIN0204_L3.6mm_D1.6mm_P1.90mm_Vertical, F.Cu at (23.9, 129.5)
- added R6: 20K, Resistor_THT:R_Axial_DIN0204_L3.6mm_D1.6mm_P1.90mm_Vertical, F.Cu at (23.9, 125.7)
- added R7: R, Resistor_THT:R_Axial_DIN0204_L3.6mm_D1.6mm_P1.90mm_Vertical, F.Cu at (42.3, 136.5)
- added R8: R, Resistor_THT:R_Axial_DIN0204_L3.6mm_D1.6mm_P1.90mm_Vertical, F.Cu at (45.5, 136.5)
- added SW1: SW_PUSH, Button_Switch_THT:SW_PUSH_6mm, F.Cu at (58.2, 142.9)
- added SW2: SW_PUSH, Button_Switch_THT:SW_PUSH_6mm, F.Cu at (69.6, 142.9)
- added U4: 74LS573, Package_DIP:DIP-20_W7.62mm, F.Cu at (106.0, 57.8)
- IC4: value 74HC273 -> 74HC697
- J2: value USB_B_Micro -> USB Module; footprint Connector_USB:USB_Micro-B_Molex_47346-0001 -> Connector_PinHeader_2.54mm:PinHeader_1x06_P2.54mm_Vertical
- U1: value 74LS377 -> 74LS245
- U16, U17, U6: value 74HC273 -> 74LS697
- moved C23 96.0 mm to (180.8, 69.2), turned to 0 degrees
- moved C14 94.0 mm to (180.8, 62.9), turned to 0 degrees
- moved C27 93.8 mm to (175.1, 78.6), turned to 0 degrees
- moved C9 90.4 mm to (175.1, 62.9), turned to 0 degrees
- moved C25 88.4 mm to (175.1, 75.5), turned to 0 degrees
- moved C11 85.8 mm to (169.5, 69.2), turned to 0 degrees
- moved U17 72.8 mm to (75.6, 119.4)
- moved U6 72.8 mm to (75.6, 108.6)
- moved IC4 72.3 mm to (75.9, 93.3)
- moved R1 72.3 mm to (107.3, 70.5)
- moved U16 72.2 mm to (75.9, 82.5)
- moved C21 70.0 mm to (169.5, 78.6), turned to 0 degrees
- moved C28 69.5 mm to (180.8, 72.3), turned to 0 degrees
- moved C5 69.2 mm to (163.8, 66.0), turned to 0 degrees
- moved C7 68.8 mm to (163.8, 69.2), turned to 0 degrees
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Connections:
- net /D/R Registers/r0 renamed Net-(U16-Pad2)
- net /D/R Registers/r1 renamed Net-(U16-Pad5)
- net /D/R Registers/r10 renamed Net-(U17-Pad6)
- net /D/R Registers/r11 renamed Net-(U17-Pad9)
- net /D/R Registers/r12 renamed Net-(U17-Pad12)
- net /D/R Registers/r13 renamed Net-(U17-Pad15)
- net /D/R Registers/r2 renamed Net-(U16-Pad6)
- net /D/R Registers/r3 renamed Net-(U16-Pad9)
- net /D/R Registers/r4 renamed Net-(U16-Pad12)
- net /D/R Registers/r8 renamed Net-(U17-Pad2)
- net /D/R Registers/r9 renamed Net-(U17-Pad5)
- net Net-(U20-Pad2) renamed /ROM/~chip_enable~
- net Net-(U20-Pad20) renamed /ROM/~output_enable~
- net Net-(U21-Pad4) renamed /Program Counter/down
- net Net-(U21-Pad5) renamed /Program Counter/up
- net Net-(U22-Pad20) renamed /RAM/~chip_enable~
- net Net-(U28-Pad20) renamed /RAM/~chip_enable
- net pc0 renamed /Program Counter/pc0
- net pc1 renamed /Program Counter/pc1
- net pc10 renamed /Program Counter/pc10
- net pc11 renamed /Program Counter/pc11
- net pc12 renamed /Program Counter/pc12
- net pc13 renamed /Program Counter/pc13
- net pc14 renamed /Program Counter/pc14
- net pc15 renamed /Program Counter/pc15
- net pc2 renamed /Program Counter/pc2
- net pc3 renamed /Program Counter/pc3
- net pc4 renamed /Program Counter/pc4
- net pc5 renamed /Program Counter/pc5
- net pc6 renamed /Program Counter/pc6
- net pc7 renamed /Program Counter/pc7
- net pc8 renamed /Program Counter/pc8
- net pc9 renamed /Program Counter/pc9
- net rom0 renamed /Program Counter/rom0
- net rom1 renamed /Program Counter/rom1
- net rom10 renamed /Program Counter/rom10
- net rom11 renamed /Program Counter/rom11
- net rom12 renamed /Program Counter/rom12
- net rom13 renamed /Program Counter/rom13
- net rom14 renamed /Program Counter/rom14
- net rom15 renamed /Program Counter/rom15
- net rom2 renamed /Program Counter/rom2
- net rom3 renamed /Program Counter/rom3
- net rom4 renamed /Program Counter/rom4
- net rom5 renamed /Program Counter/rom5
- net rom6 renamed /Program Counter/rom6
- net rom7 renamed /Program Counter/rom7
- net rom8 renamed /Program Counter/rom8
- net rom9 renamed /Program Counter/rom9
- net stack_a8 renamed /Stack/a8
- net tos0 renamed /ADD/tos0
- net tos1 renamed /ADD/tos1
- net tos10 renamed /ADD/tos10
- net tos11 renamed /ADD/tos11
- net tos12 renamed /ADD/tos12
- net tos13 renamed /ADD/tos13
- net tos14 renamed /ADD/tos14
- net tos15 renamed /ADD/tos15
- net tos2 renamed /ADD/tos2
- net tos3 renamed /ADD/tos3
- net tos4 renamed /ADD/tos4
- net tos5 renamed /ADD/tos5
- net tos6 renamed /ADD/tos6
- net tos7 renamed /ADD/tos7
- net tos8 renamed /ADD/tos8
- net tos9 renamed /ADD/tos9
- net tos_bus0 renamed /ADD/tos_bus0
- net tos_bus1 renamed /ADD/tos_bus1
- net tos_bus10 renamed /ADD/tos_bus10
- net tos_bus11 renamed /ADD/tos_bus11
- net tos_bus12 renamed /ADD/tos_bus12
- net tos_bus13 renamed /ADD/tos_bus13
- net tos_bus14 renamed /ADD/tos_bus14
- net tos_bus15 renamed /ADD/tos_bus15
- net tos_bus2 renamed /ADD/tos_bus2
- net tos_bus3 renamed /ADD/tos_bus3
- net tos_bus4 renamed /ADD/tos_bus4
- net tos_bus5 renamed /ADD/tos_bus5
- net tos_bus6 renamed /ADD/tos_bus6
- net tos_bus7 renamed /ADD/tos_bus7
- net tos_bus8 renamed /ADD/tos_bus8
- net tos_bus9 renamed /ADD/tos_bus9
- C4 pad 1: GNDREF -> VCC
- C4 pad 2: VCC -> GNDREF
- C8 pad 1: VCC -> GNDREF
- C8 pad 2: GNDREF -> VCC
- IC4 pad 12: stack4 -> Net-(IC4-Pad12)
- IC4 pad 13: Net-(IC4-Pad13) -> VCC
- IC4 pad 15: stack5 -> Net-(IC4-Pad15)
- IC4 pad 16: stack6 -> /D/R Registers/stack2
- IC4 pad 17: Net-(IC4-Pad17) -> /D/R Registers/stack1
- IC4 pad 18: Net-(IC4-Pad18) -> /D/R Registers/stack0
- IC4 pad 19: stack7 -> (no net)
- IC4 pad 2: stack0 -> Net-(IC4-Pad2)
- IC4 pad 5: stack1 -> Net-(IC4-Pad5)
- IC4 pad 6: stack2 -> Net-(IC4-Pad6)
- IC4 pad 7: Net-(IC4-Pad7) -> /D/R Registers/~d_enable
- IC4 pad 9: stack3 -> Net-(IC4-Pad9)
- J2 pad 1: Net-(J2-Pad1) -> VCC
- J2 pad 2: Net-(J2-Pad2) -> GNDREF
- R1 pad 2: jump0 -> /JUMP / CHAR/jump0
- U1 pad 10: Net-(U1-Pad10) -> GNDREF
- U1 pad 11: Net-(U1-Pad11) -> Net-(J1-Pad6)
- U1 pad 12: Net-(J1-Pad12) -> Net-(J1-Pad8)
- U1 pad 13: Net-(U1-Pad13) -> Net-(J1-Pad10)
- U1 pad 14: Net-(U1-Pad14) -> Net-(J1-Pad12)
- U1 pad 15: Net-(J1-Pad10) -> Net-(J1-Pad5)
- U1 pad 16: Net-(J1-Pad8) -> Net-(J1-Pad7)
- U1 pad 17: Net-(U1-Pad17) -> Net-(J1-Pad9)
- U1 pad 18: Net-(U1-Pad18) -> Net-(J1-Pad11)
- U1 pad 19: Net-(J1-Pad6) -> Net-(U1-Pad19)
- U1 pad 2: Net-(J1-Pad11) -> /ADD/stack0
- U1 pad 20: Net-(U1-Pad20) -> VCC
- U1 pad 3: Net-(U1-Pad3) -> /ADD/stack1
- U1 pad 4: Net-(U1-Pad4) -> /ADD/stack2
- U1 pad 5: Net-(J1-Pad9) -> /ADD/stack3
- U1 pad 6: Net-(J1-Pad7) -> /ADD/stack4
- U1 pad 7: Net-(U1-Pad7) -> /ADD/stack5
- U1 pad 8: Net-(U1-Pad8) -> /ADD/stack6
- U1 pad 9: Net-(J1-Pad5) -> /ADD/stack7
- U10 pad 1: stack7 -> /D/R Registers/stack7
- U10 pad 10: stack_bus1 -> /ADD/stack1
- U10 pad 11: stack_bus2 -> /ADD/stack2
- U10 pad 12: Net-(U10-Pad12) -> GNDREF
- U10 pad 13: stack_bus3 -> /ADD/stack3
- U10 pad 14: stack_bus4 -> /ADD/stack4
- U10 pad 15: stack_bus5 -> /ADD/stack5
- U10 pad 16: stack_bus6 -> /ADD/stack6
- U10 pad 17: stack_bus7 -> /ADD/stack7
- U10 pad 2: stack6 -> /D/R Registers/stack6
- U10 pad 24: Net-(U10-Pad24) -> VCC
- U10 pad 3: stack5 -> /D/R Registers/stack5
- U10 pad 4: stack4 -> /D/R Registers/stack4
- U10 pad 5: stack3 -> /D/R Registers/stack3
- U10 pad 6: stack2 -> /D/R Registers/stack2
- U10 pad 7: stack1 -> /D/R Registers/stack1
- U10 pad 8: stack0 -> /D/R Registers/stack0
- U10 pad 9: stack_bus0 -> /ADD/stack0
- U11 pad 1: stack15 -> /D/R Registers/stack7
- U11 pad 10: stack_bus9 -> /ADD/stack9
- U11 pad 11: stack_bus10 -> /ADD/stack10
- U11 pad 12: Net-(U11-Pad12) -> GNDREF
- U11 pad 13: stack_bus11 -> /ADD/stack11
- U11 pad 14: stack_bus12 -> /ADD/stack12
- U11 pad 15: stack_bus13 -> /ADD/stack13
- U11 pad 16: stack_bus14 -> /ADD/stack14
- U11 pad 17: stack_bus15 -> /ADD/stack15
- U11 pad 2: stack14 -> /D/R Registers/stack6
- U11 pad 24: Net-(U11-Pad24) -> VCC
- U11 pad 3: stack13 -> /D/R Registers/stack5
- U11 pad 4: stack12 -> /D/R Registers/stack4
- U11 pad 5: stack11 -> /D/R Registers/stack3
- U11 pad 6: stack10 -> /D/R Registers/stack2
- U11 pad 7: stack9 -> /D/R Registers/stack1
- U11 pad 8: stack8 -> /D/R Registers/stack0
- U11 pad 9: stack_bus8 -> /ADD/stack8
- U12 pad 11: stack3 -> /ADD/stack3
- U12 pad 15: stack2 -> /ADD/stack2
- U12 pad 16: VCC -> /ADD/enable
- U12 pad 2: stack1 -> /ADD/stack1
- U12 pad 6: stack0 -> /ADD/stack0
- U12 pad 7: Net-(U12-Pad7) -> GNDREF
- U13 pad 11: stack7 -> /ADD/stack7
- U13 pad 15: stack6 -> /ADD/stack6
- U13 pad 16: VCC -> /ADD/enable
- U13 pad 2: stack5 -> /ADD/stack5
- U13 pad 6: stack4 -> /ADD/stack4
- U14 pad 10: stack10 -> /ADD/stack10
- U14 pad 13: stack11 -> /ADD/stack11
- U14 pad 14: VCC -> /NAND/enable
- U14 pad 2: stack8 -> /ADD/stack8
- U14 pad 5: stack9 -> /ADD/stack9
- U15 pad 10: stack14 -> /ADD/stack14
- U15 pad 13: stack15 -> /ADD/stack15
- U15 pad 14: VCC -> /NAND/enable
- U15 pad 2: stack12 -> /ADD/stack12
- U15 pad 5: stack13 -> /ADD/stack13
- U16 pad 10: GNDREF -> Net-(U16-Pad10)
- U16 pad 13: Net-(U16-Pad13) -> VCC
- U16 pad 15: /D/R Registers/r5 -> Net-(U16-Pad15)
- U16 pad 16: /D/R Registers/r6 -> /D/R Registers/stack2
- U16 pad 17: Net-(U16-Pad17) -> /D/R Registers/stack1
- U16 pad 18: Net-(U16-Pad18) -> /D/R Registers/stack0
- U16 pad 19: /D/R Registers/r7 -> (no net)
- U16 pad 7: Net-(U16-Pad7) -> /D/R Registers/~r_enable
- U17 pad 13: Net-(U17-Pad13) -> VCC
- U17 pad 14: Net-(U17-Pad14) -> Net-(U16-Pad15)
- U17 pad 16: /D/R Registers/r14 -> /D/R Registers/stack6
- U17 pad 17: Net-(U17-Pad17) -> /D/R Registers/stack5
- U17 pad 18: Net-(U17-Pad18) -> /D/R Registers/stack4
- U17 pad 19: /D/R Registers/r15 -> (no net)
- U17 pad 7: Net-(U17-Pad7) -> /D/R Registers/~r_enable
- U18 pad 11: stack11 -> /ADD/stack11
- U18 pad 15: stack10 -> /ADD/stack10
- U18 pad 16: VCC -> /ADD/enable
- U18 pad 2: stack9 -> /ADD/stack9
- U18 pad 6: stack8 -> /ADD/stack8
- U19 pad 11: stack15 -> /ADD/stack15
- U19 pad 15: stack14 -> /ADD/stack14
- U19 pad 16: VCC -> /ADD/enable
- U19 pad 2: stack13 -> /ADD/stack13
- U19 pad 6: stack12 -> /ADD/stack12
- U2 pad 10: stack2 -> /ADD/stack2
- U2 pad 13: stack3 -> /ADD/stack3
- U2 pad 14: VCC -> /NAND/enable
- U2 pad 2: stack0 -> /ADD/stack0
- U2 pad 5: stack1 -> /ADD/stack1
- U21 pad 11: Net-(U21-Pad11) -> /JUMP / CHAR/jump0
- U21 pad 14: Net-(U21-Pad14) -> GNDREF
- U22 pad 1: ram5 -> /ADD/stack5
- U22 pad 10: ram14 -> /ADD/stack14
- U22 pad 2: ram6 -> /ADD/stack6
- U22 pad 21: ram0 -> /ADD/stack0
- U22 pad 22: Net-(U22-Pad22) -> /RAM/~output_enable~
- U22 pad 23: ram1 -> /ADD/stack1
- U22 pad 24: ram2 -> /ADD/stack2
- U22 pad 25: ram3 -> /ADD/stack3
- U22 pad 26: ram4 -> /ADD/stack4
- U22 pad 27: Net-(U22-Pad27) -> /RAM/~write_enable~
- U22 pad 3: ram7 -> /ADD/stack7
- U22 pad 4: ram8 -> /ADD/stack8
- U22 pad 5: ram9 -> /ADD/stack9
- U22 pad 6: ram10 -> /ADD/stack10
- U22 pad 7: ram11 -> /ADD/stack11
- U22 pad 8: ram12 -> /ADD/stack12
- U22 pad 9: ram13 -> /ADD/stack13
- U23 pad 11: Net-(U23-Pad11) -> /JUMP / CHAR/jump0
- U23 pad 14: Net-(U23-Pad14) -> GNDREF
- U23 pad 4: Net-(U23-Pad4) -> GNDREF
- U24 pad 11: Net-(U24-Pad11) -> /JUMP / CHAR/jump0
- U24 pad 14: Net-(U24-Pad14) -> GNDREF
- U24 pad 4: Net-(U24-Pad4) -> GNDREF
- U24 pad 5: Net-(U24-Pad5) -> Net-(U21-Pad12)
- U25 pad 11: Net-(U25-Pad11) -> /JUMP / CHAR/jump0
- U25 pad 12: Net-(U25-Pad12) -> Net-(U23-Pad5)
- U25 pad 14: Net-(U25-Pad14) -> GNDREF
- U25 pad 4: Net-(U25-Pad4) -> GNDREF
- U25 pad 5: Net-(U25-Pad5) -> Net-(U24-Pad12)
- U28 pad 22: Net-(U28-Pad22) -> /RAM/~output_enable~
- U28 pad 27: Net-(U28-Pad27) -> /RAM/~write_enable~
- U3 pad 10: stack6 -> /ADD/stack6
- U3 pad 13: stack7 -> /ADD/stack7
- U3 pad 14: VCC -> /NAND/enable
- U3 pad 2: stack4 -> /ADD/stack4
- U3 pad 5: stack5 -> /ADD/stack5
- U6 pad 12: stack12 -> Net-(U6-Pad12)
- U6 pad 13: Net-(U6-Pad13) -> VCC
- U6 pad 14: Net-(U6-Pad14) -> Net-(IC4-Pad15)
- U6 pad 15: stack13 -> Net-(U6-Pad15)
- U6 pad 16: stack14 -> /D/R Registers/stack6
- U6 pad 17: Net-(U6-Pad17) -> /D/R Registers/stack5
- U6 pad 18: Net-(U6-Pad18) -> /D/R Registers/stack4
- U6 pad 19: stack15 -> (no net)
- U6 pad 2: stack8 -> Net-(U6-Pad2)
- U6 pad 5: stack9 -> Net-(U6-Pad5)
- U6 pad 6: stack10 -> Net-(U6-Pad6)
- U6 pad 7: Net-(U6-Pad7) -> /D/R Registers/~d_enable
- U6 pad 9: stack11 -> Net-(U6-Pad9)
- U8 pad 3: /Clock/CLK -> /Power/Clock/clk
Routing:
- net VCC: track 0.00 -> 16.9 mm
- net /D/R Registers/stack2: track 0.00 -> 14.3 mm
- net /D/R Registers/stack4: track 0.00 -> 14.0 mm
- net /D/R Registers/stack5: track 0.00 -> 14.0 mm
- net /D/R Registers/stack3: track 0.00 -> 14.0 mm
- net /Stack/a8: track 0.00 -> 14.0 mm
- net /D/R Registers/stack7: track 0.00 -> 14.0 mm
- net /D/R Registers/stack6: track 0.00 -> 14.0 mm
- net /D/R Registers/stack1: track 0.00 -> 14.0 mm
- net /D/R Registers/stack0: track 0.00 -> 14.0 mm
- net GNDREF: track 4.78 -> 0.00 mm
- net Net-(U5-Pad10): track 0.00 -> 1.86 mm
Other:
- board text added: "ADD [74HCT283]"
- board text added: "CLK [555]"
- board text added: "CTRL [74HCT573]"
- board text added: "D [74LS697]"
- board text added: "I/O [74HCT245]"
- board text added: "NAND [74HCT00]"
- board text added: "PROGRAM COUNTER [74HCT193]"
- board text added: "R [74LS697]"
- board text added: "RAM (32K) [CY62256]"
- board text added: "RESET"
- board text added: "ROM (32K) [27C1024]"
- board text added: "STACK (2K) [CY6116]"
- board text added: "STEP"
- board text added: "TOM-1 Board Schematic"
- board text added: "TOS [74HCT377]"
- board text added: "TTL OPERATION MODULE"
- board text removed: "ADD"
- board text removed: "CLOCK"
- board text removed: "D REGISTER"
- board text removed: "DECODE"
- board text removed: "I/O REGISTER"
- board text removed: "NAND"
- board text removed: "PROGRAM COUNTER"
- board text removed: "R REGISTER"
- board text removed: "RAM (32K)"
- board text removed: "ROM (32K)"
- board text removed: "STACK (256×2)"
- board text removed: "TOS REGISTER"
- board text removed: "TTL"
- board text removed: "TTL OPERATION MODULE (TOM-1)"

Commit message: Initial commit
Parts:
- added D2: LED, LED_THT:LED_D3.0mm, F.Cu at (125.1, 138.4)
- added R9: R, Resistor_THT:R_Axial_DIN0204_L3.6mm_D1.6mm_P1.90mm_Vertical, F.Cu at (125.7, 143.5)
- moved C9 129.5 mm to (45.7, 57.1), turned to 90 degrees
- moved C11 123.8 mm to (45.7, 67.9), turned to 90 degrees
- moved C4 122.1 mm to (45.7, 31.7), turned to 90 degrees
- moved C5 120.5 mm to (45.7, 41.9), turned to 90 degrees
- moved C10 119.2 mm to (45.7, 88.2), turned to 90 degrees
- moved C7 118.4 mm to (45.7, 78.1), turned to 90 degrees
- moved C19 113.0 mm to (69.8, 128.9), turned to 90 degrees
- moved C14 111.1 mm to (69.8, 57.1), turned to 90 degrees
- moved C18 110.9 mm to (69.8, 67.9), turned to 90 degrees
- moved C27 110.2 mm to (69.8, 111.1), turned to 90 degrees
- moved C23 109.6 mm to (99.1, 142.2), turned to 90 degrees
- moved C12 107.9 mm to (69.8, 89.5), turned to 90 degrees
- moved C17 105.7 mm to (69.8, 78.7), turned to 90 degrees
- moved C6 103.8 mm to (70.5, 31.8), turned to 90 degrees
- moved C8 101.9 mm to (70.5, 41.9), turned to 90 degrees
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- renumbered A8 to PGM1
Connections:
- IC7 pad 1: Net-(IC7-Pad1) -> /TOS/~clock_enable
- IC7 pad 11: Net-(IC7-Pad11) -> /TOS/clk
- IC9 pad 1: Net-(IC9-Pad1) -> /TOS/~clock_enable
- IC9 pad 11: Net-(IC9-Pad11) -> /TOS/clk
- Q1 pad 1: /Power/Clock/clk_bar -> /TOS/clk
- R8 pad 2: /Power/Clock/clk_bar -> /TOS/clk
- U10 pad 18: Net-(U10-Pad18) -> /Stack/~chip_select
- U10 pad 19: Net-(U10-Pad19) -> GNDREF
- U10 pad 20: Net-(U10-Pad20) -> /Stack/~output_enable
- U10 pad 21: Net-(U10-Pad21) -> /Stack/~write_enable
- U10 pad 22: Net-(U10-Pad22) -> GNDREF
- U11 pad 18: Net-(U11-Pad18) -> /Stack/~chip_select
- U11 pad 19: Net-(U11-Pad19) -> GNDREF
- U11 pad 20: Net-(U11-Pad20) -> /Stack/~output_enable
- U11 pad 21: Net-(U11-Pad21) -> /Stack/~write_enable
- U11 pad 22: Net-(U11-Pad22) -> GNDREF
- U21 pad 4: /Program Counter/down -> GNDREF
- U4 pad 11: /Power/Clock/clk_bar -> /TOS/clk
Routing:
- net /ADD/stack6: track 0.00 -> 136.0 mm, vias 0 -> 1
- net /ADD/stack5: track 0.00 -> 122.0 mm, vias 0 -> 1
- net /ADD/stack7: track 0.00 -> 103.0 mm
- net /ADD/stack2: track 0.00 -> 91.3 mm, vias 0 -> 1
- net /ADD/stack3: track 0.00 -> 62.2 mm, vias 0 -> 2
- net /ADD/stack4: track 0.00 -> 61.4 mm, vias 0 -> 1
- net /ADD/tos0: track 0.00 -> 50.8 mm
- net /ADD/tos14: track 0.00 -> 46.2 mm
- net /ADD/tos15: track 0.00 -> 42.1 mm
- net /D/R Registers/stack4: track 14.0 -> 54.2 mm
- net /D/R Registers/stack5: track 14.0 -> 52.2 mm
- net /ADD/tos7: track 0.00 -> 38.0 mm
- net Net-(U16-Pad15): track 0.00 -> 37.4 mm
- net /D/R Registers/~r_enable: track 0.00 -> 37.3 mm
- net GND: track 0.00 -> 36.6 mm
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
Commit message: Lots of Digital work
Other:
- board text added: "PROGRAM COUNTER [74HCT191]"
- board text added: "TOS [74HCT273]"
- board text removed: "PROGRAM COUNTER [74HCT193]"
- board text removed: "TOS [74HCT377]"
